File: PCB files/Phantom/Phantom.kicad_sch (KiCad schematic)
At the start: 24 parts, among them J1 Micro_SD_Card, J2 USB_B_Micro, J3 Conn_01x02_Socket, SW1 SW_Push, SW2 SW_Push, U1 ESP32-S3-MINI-1, U2 MAX-M10S, U3 D3V3XA4B10LP, U5 TLV76733DRVx, U6 MCP73871-2CC

Commit message: Schematic work
Parts:
- removed J1: Micro_SD_Card, symbol Connector:Micro_SD_Card
- removed U4: ~, symbol LS027 LCD:SHARP_LCD
- added BT1: Battery_Cell, BC501SM:BAT_BC501SM, symbol Device:Battery_Cell
- added C10: 100n, Capacitor_SMD:C_0603_1608Metric, symbol Device:C
- added C11: 10u, symbol Device:C
- added C7, C8: 100n, Capacitor_SMD:C_0201_0603Metric, symbol Device:C
- added C9: 1u, symbol Device:C
- added J1: MEM2052-00-195-00-A_REVA, MEM2052_00_195_00_A:GCT_MEM2052-00-195-00-A_REVA, symbol MEM2052-00-195-00-A_REVA:MEM2052-00-195-00-A_REVA
- added J4: Conn_Coaxial, symbol Connector:Conn_Coaxial
- added L1: L, symbol Device:L
- added R10, R11, R7, R8, R9: 10k, Resistor_SMD:R_0603_1608Metric, symbol Device:R
- added R12: 10, Resistor_SMD:R_0603_1608Metric, symbol Device:R
- added U7: ~, symbol LS027 LCD:SHARP_LCD
- C1, C3, C4: footprint (none) -> Capacitor_SMD:C_0603_1608Metric
- R1, R2, R3, R4, R5, R6, TH1: footprint (none) -> Resistor_SMD:R_0603_1608Metric
- SW1, SW2: footprint (none) -> B3U_1100P:SW_B3U-1100P
Connections:
- net +3.3V: now also U2.7 (VCC_IO), U2.8 (VCC), C7.1, C8.1, C9.1, J1.P4 (VDD), R10.1, R11.1, R7.1, R8.1, R9.1, U7.6 (VDDA), U7.7 (VDD), U7.8 (EXTMODE)
- net GND: now also U2.1 (GND), U2.10 (GND), U2.12 (GND), BT1.2 (-), C10.2, C11.2, C7.2, C8.2, C9.2, J1.G1 (SHIELD_GND), J1.G2 (SHIELD_GND__1), J1.G3 (SHIELD_GND__2), J1.G4 (SHIELD_GND__3), J1.P6 (VSS), J4.2 (Ext), U7.10 (VSSA), U7.9 (VSS)
- net STAT2: now also U1.44 (IO46); no longer U1.41 (IO45)
- net VBUS: now also C11.1
- net DAT2: now reaches U1.10 (IO6)
- net DAT2: now also J1.P1 (DAT2), R10.2
- net DAT3: now reaches U1.11 (IO7)
- net DAT3: now also J1.P2 (CD/DAT3), R9.2
- net CD_PIN: now reaches U1.12 (IO8)
- net CD_PIN: now also J1.P9 (CD_PIN)
- net SCS: now reaches U1.14 (IO10)
- net SCS: now also U1.26 (IO26), U7.3 (SCS)
- net SI: now reaches U1.28 (IO33)
- net SI: now also U7.2 (SI)
- net SCLK: now reaches U1.29 (IO34)
- net SCLK: now also U7.1 (SCLK)
- net DISPCNTRL: now reaches U1.31 (IO35)
- net DISPCNTRL: now also C10.1, U7.5 (DISP)
- net EXTCOMIN: now reaches U1.34 (IO38)
- net EXTCOMIN: now also U7.4 (EXTCOMIN)
- net GPSRX: now reaches U1.39 (TXD0)
- net GPSRX: now also U2.3 (RXD)
- net GPSTX: now reaches U1.40 (RXD0)
- net GPSTX: now also U2.2 (TXD)
- net CLK: now reaches U1.5 (IO1)
- net CLK: now also J1.P5 (CLK)
- net CMD: now reaches U1.6 (IO2)
- net CMD: now also J1.P3 (CMD), R8.2
- net DAT0: now reaches U1.8 (IO4)
- net DAT0: now also J1.P7 (DAT0), R7.2
- net DAT1: now reaches U1.9 (IO5)
- net DAT1: now also J1.P8 (DAT1), R11.2
- net at U2.11 (RF_IN): now also J4.1 (In), L1.2
- net at U2.14 (VCC_RF): now also L1.1
- net at U2.6 (V_BCKP): now also R12.2
- new net: BT1.1 (+), R12.1
Other:
- moved on the sheet: U2

Commit message: Finished PCB and starting CAD
Parts:
- added C12, C13, C15: 100n, Capacitor_SMD:C_0603_1608Metric, symbol Device:C
- added C14: 2.2u, Capacitor_SMD:C_0603_1608Metric, symbol Device:C
- added H1, H2, H3, H4: MountingHole, MountingHole:MountingHole_3.2mm_M3, symbol Mechanical:MountingHole
- added R13, R14, R15, R16: 10k, Resistor_SMD:R_0603_1608Metric, symbol Device:R
- added R17, R18: 0, Resistor_SMD:R_0603_1608Metric, symbol Device:R
- added SW3: RotaryEncoder_Switch, footprintsconn:COM-15141_SPK, symbol Device:RotaryEncoder_Switch
- added SW4: SW_SPST, footprintsSPST:SW_1MS02Q_CNK, symbol Switch:SW_SPST
- C11, C2: footprint (none) -> Capacitor_SMD:C_0805_2012Metric
- C5, C6, C9: footprint (none) -> Capacitor_SMD:C_0603_1608Metric
- C7, C8: footprint Capacitor_SMD:C_0201_0603Metric -> Capacitor_SMD:C_0603_1608Metric
- J2: footprint (none) -> DX4R005HJ5R2000:JAE_DX4R005HJ5R2000
- J3: footprint (none) -> Connector_JST:JST_PH_S2B-PH-K_1x02_P2.00mm_Horizontal
- J4: footprint (none) -> Connector_Coaxial:U.FL_Hirose_U.FL-R-SMT-1_Vertical
- L1: value L -> 47n; footprint (none) -> Inductor_SMD:L_0603_1608Metric
- U1: footprint RF_Module:ESP32-S2-MINI-1 -> foot:ESP32-S3-MINI-1_EXP
- U7: footprint (none) -> FH33_10S_0_5SH_10_:HRS_FH33-10S-0.5SH_10_
Connections:
- net +3.3V: now also C14.2, C15.2, R13.2, R14.2, R15.2, R16.1
- net CD_PIN: now also U1.18 (IO14), R16.2; no longer U1.12 (IO8)
- net CLK: now also U1.19 (IO15); no longer U1.5 (IO1)
- net CMD: now also U1.20 (IO16); no longer U1.6 (IO2)
- net D+: now also R18.2; no longer U1.24 (USB_D+)
- net D-: now also R17.2; no longer U1.23 (USB_D-)
- net DAT0: now also U1.16 (IO12); no longer U1.8 (IO4)
- net DAT1: now also U1.17 (IO13); no longer U1.9 (IO5)
- net DAT2: now also U1.22 (IO18); no longer U1.10 (IO6)
- net DAT3: now also U1.21 (IO17); no longer U1.11 (IO7)
- net DISPCNTRL: now also U1.35 (IO39); no longer U1.31 (IO35)
- net GND: now also C12.2, C13.2, C14.1, C15.1, SW3.C, SW3.S2
- net LDOIN: now also SW4.2 (B); no longer U6.1 (OUT), U6.20 (OUT)
- net PG: now also U1.11 (IO7); no longer U1.27 (IO47)
- net SCLK: now also U1.31 (IO35); no longer U1.29 (IO34)
- net SCS: now also U1.33 (IO37); no longer U1.14 (IO10), U1.26 (IO26)
- net SI: now also U1.32 (IO36); no longer U1.28 (IO33)
- net STAT1: now also U1.9 (IO5); no longer U1.37 (IO41)
- net STAT2: now also U1.10 (IO6); no longer U1.44 (IO46)
- net VBCK: now reaches R12.2, U2.6 (V_BCKP)
- net A: now reaches U1.13 (IO9)
- net A: now also C13.1, R14.1, SW3.A
- net B: now reaches U1.15 (IO11)
- net B: now also C12.1, R13.1, SW3.B
- new net 1D-: R17.1, U1.23 (USB_D-)
- new net 2D+: R18.1, U1.24 (USB_D+)
- new net OUT: SW4.1 (A), U6.1 (OUT), U6.20 (OUT)
- new net S1: R15.1, SW3.S1, U1.14 (IO10)
Other:
- moved on the sheet: BT1, C10, C11, C7, C8, C9, J1, J3, J4, L1, R10, R11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

Commit message: PCB Fix
Other:
- note added: "Battery Charging"
- note added: "Display"
- note added: "ESP32"
- note added: "GPS"
- note added: "Rotary Encoder"
- note added: "SD Card"
- moved on the sheet: BT1, C10, C12, C13, C14, C15, C7, C8, C9, H1, H2, H3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
